File: hardware/pcb/QUADRUPED_ROBOT/mach_robot.kicad_pcb (KiCad board)
At the start: 2 copper layers, 100 x 100 mm, 164 parts, among them J1 Conn_01x03_Socket, J10 PIN, J11 Conn_01x03_Pin, J12 Conn_01x03_Pin, J13 Conn_01x03_Pin, J14 Conn_01x03_Pin, J15 Conn_01x03_Pin, J16 Conn_01x03_Pin, J17 Conn_01x03_Pin, J18 Conn_01x03_Pin, J19 Conn_01x03_Pin, J2 Conn_01x04_Pin, J20 Conn_01x03_Pin, J21 Conn_01x03_Pin, J22 Conn_01x03_Pin, J3 SWITCH_POWER, J5 PIN, J6 USB_C_Receptacle_USB2.0_16P, J7 USB_A, J8 Conn_01x06_Pin, J9 JETSON, Q1 AO4485, Q2 BC847, Q3 BC847, SW1 SW_Push, U1 XL4016, U2 STM32F723ZETx, U3 TPS5430DDA, U4 USBLC6-2SC6, Y1 25MHz

Commit message: pcb update
Parts:
- added C64: 100nF, Capacitor_SMD:C_0805_2012Metric, F.Cu at (97.8, 82.7)
- added J4: Conn_01x03_Pin, Connector_PinHeader_2.54mm:PinHeader_1x03_P2.54mm_Vertical, F.Cu at (71.3, 91.4)
- added R5: 10m, Resistor_SMD:R_2512_6332Metric, B.Cu at (86.7, 92.2)
- added R50: 10K, Resistor_SMD:R_0805_2012Metric, B.Cu at (86.4, 86.4)
- added R51: 10K, Resistor_SMD:R_0805_2012Metric, B.Cu at (85.1, 85.1)
- added R52: 10K, Resistor_SMD:R_0805_2012Metric, F.Cu at (86.3, 79.7)
- added R59: 10K, Resistor_SMD:R_0805_2012Metric, B.Cu at (93.0, 90.9)
- added R61: 4.7K, Resistor_SMD:R_0805_2012Metric, F.Cu at (89.7, 75.3)
- added R62: 10K, Resistor_SMD:R_0805_2012Metric, F.Cu at (91.1, 76.7)
- added R63: 30K, Resistor_SMD:R_0805_2012Metric, F.Cu at (92.5, 78.1)
- added R64: 4.7K, Resistor_SMD:R_0805_2012Metric, F.Cu at (84.9, 78.3)
- added R7: 50m, Resistor_SMD:R_2512_6332Metric, B.Cu at (98.4, 90.0)
- added R8: 10m, Resistor_SMD:R_2512_6332Metric, B.Cu at (103.0, 81.8)
- added U5: INA3221, Package_DFN_QFN:Texas_RGV0016A_VQFN-16-1EP_4x4mm_P0.65mm_EP2.1x2.1mm, F.Cu at (92.5, 83.1)
- moved R1 1.33 mm to (102.3, 72.4)
- moved C1 1.33 mm to (99.9, 75.6)
- moved C2 1.33 mm to (103.8, 73.9)
- moved Y1 1.33 mm to (100.0, 68.8)
- moved R2 0.62 mm to (84.8, 74.3)
Connections:
- net +6V renamed +6V_SERVO
- net Net-(F1-Pad2) renamed /power supply/IN_+1
- C34 pad 2: Net-(D5-A2) -> +5V_P
- D5 pad 2: Net-(D5-A2) -> +5V_P
- F2 pad 1: Net-(D5-A2) -> +5V_P
- J7 pad 1: Net-(D5-A2) -> +5V_P
- R43 pad 1: Net-(D5-A2) -> +5V_P
- U2 pad 10: unconnected-(U2-PF0-Pad10) -> /chip/SDA
- U2 pad 11: unconnected-(U2-PF1-Pad11) -> /chip/SCL
- U2 pad 13: unconnected-(U2-PF3-Pad13) -> Net-(U2-PF3)
- U2 pad 142: unconnected-(U2-PE1-Pad142) -> /chip/WRN
Routing:
- net +5V_P: track 99.0 -> 297.7 mm, vias 0 -> 3
- net +6V_SERVO: track 319.5 -> 397.0 mm, vias 1 -> 3
- net +12V: track 117.9 -> 194.3 mm, vias 0 -> 3
- net +3.3V: track 350.7 -> 421.6 mm, vias 8 -> 10
- net Net-(D5-A2): track 47.3 -> 0.00 mm
- net /power supply/IN_+1: track 23.2 -> 61.6 mm, vias 0 -> 1
- net /chip/WRN: track 0.00 -> 25.6 mm
- net /chip/SCL: track 0.00 -> 20.6 mm
- net /chip/SDA: track 0.00 -> 20.2 mm
- net Net-(U2-PF3): track 0.00 -> 12.9 mm
- net Net-(U5-TC): track 0.00 -> 6.83 mm, vias 0 -> 1
- net Net-(U5-CRITICAL): track 0.00 -> 5.79 mm, vias 0 -> 1
- net Net-(U5-PV): track 0.00 -> 4.52 mm, vias 0 -> 1
- net GND: track 102.8 -> 105.7 mm, vias 55 -> 61
- net /chip/OSC_IN: track 15.6 -> 13.4 mm
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