File: hardware/pcb/QUADRUPED_ROBOT/mach_robot.kicad_sch (KiCad schematic)
At the start: 0 parts

Commit message: pcb update
Other:
- sheet chip ports: added SCL, SDA, WRN; removed none
- sheet power supply ports: added SCL, SDA, WRN; removed none
Changed lines of the file:
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@@
+	(wire
+		(pts
+			(xy 132.08 46.99) (xy 132.08 33.02)
+		)
+		(stroke
+			(width 0)
+			(type default)
+		)
+	)
 	(wire
 		(pts
@@
 	(wire
 		(pts
+			(xy 214.63 59.69) (xy 238.76 59.69)
+		)
+		(stroke
+			(width 0)
+			(type default)
+		)
+	)
+	(wire
+		(pts
 			(xy 105.41 104.14) (xy 110.49 104.14)
 		)
@@
 	(wire
 		(pts
+			(xy 111.76 43.18) (xy 125.73 43.18)
+		)
+		(stroke
+			(width 0)
+			(type default)
+		)
+	)
+	(wire
+		(pts
 			(xy 109.22 99.06) (xy 115.57 99.06)
 		)
@@
 	(wire
 		(pts
+			(xy 220.98 54.61) (xy 238.76 54.61)
+		)
+		(stroke
+			(width 0)
+			(type default)
+		)
+	)
+	(wire
+		(pts
 			(xy 110.49 104.14) (xy 110.49 149.86)
 		)
@@
 	(wire
 		(pts
+			(xy 121.92 20.32) (xy 220.98 20.32)
+		)
+		(stroke
+			(width 0)
+			(type default)
+		)
+	)
+	(wire
+		(pts
 			(xy 105.41 106.68) (xy 105.41 149.86)
 		)
@@
 	(wire
 		(pts
+			(xy 214.63 27.94) (xy 214.63 59.69)
+		)
+		(stroke
+			(width 0)
+			(type default)
+		)
+	)
+	(wire
+		(pts
+			(xy 125.73 27.94) (xy 214.63 27.94)
+		)
+		(stroke
+			(width 0)
+			(type default)
+		)
+	)
+	(wire
+		(pts
+			(xy 121.92 38.1) (xy 121.92 20.32)
+		)
+		(stroke
+			(width 0)
+			(type default)
+		)
+	)
+	(wire
+		(pts
 			(xy 111.76 78.74) (xy 115.57 78.74)
 		)
@@
 	(wire
 		(pts
+			(xy 111.76 38.1) (xy 121.92 38.1)
+		)
+		(stroke
+			(width 0)
+			(type default)
+		)
+	)
+	(wire
+		(pts
 			(xy 123.19 86.36) (xy 130.81 86.36)
 		)
@@
 	(wire
 		(pts
+			(xy 125.73 43.18) (xy 125.73 27.94)
+		)
+		(stroke
+			(width 0)
+			(type default)
+		)
+	)
+	(wire
+		(pts
 			(xy 80.01 119.38) (xy 82.55 119.38)
 		)
@@
 	(wire
 		(pts
+			(xy 132.08 33.02) (xy 207.01 33.02)
+		)
+		(stroke
+			(width 0)
+			(type default)
+		)
+	)
+	(wire
+		(pts
 			(xy 120.65 96.52) (xy 120.65 149.86)
 		)
@@
 		)
 	)
+	(wire
+		(pts
+			(xy 220.98 20.32) (xy 220.98 54.61)
+		)
+		(stroke
+			(width 0)
+			(type default)
+		)
+	)
+	(wire
+		(pts
+			(xy 207.01 33.02) (xy 207.01 66.04)
+		)
+		(stroke
+			(width 0)
+			(type default)
+		)
+	)
+	(wire
+		(pts
+			(xy 207.01 66.04) (xy 238.76 66.04)
+		)
+		(stroke
+			(width 0)
+			(type default)
+		)
+	)
+	(wire
+		(pts
+			(xy 111.76 46.99) (xy 132.08 46.99)
+		)
+		(stroke
+			(width 0)
+			(type default)
+		)
+	)
 	(sheet
-		(at 140.97 36.83)
+		(at 236.474 150.876)
 		(size 59.69 48.26)
 		(exclude_from_sim no)
@@
 		)
 		(property "Sheetname" "usb"
-			(at 140.97 36.1184 0)
+			(at 236.474 150.1644 0)
 			(show_name no)
 			(do_not_autoplace no)
@@
 		)
 		(property "Sheetfile" "usb.kicad_sch"
-			(at 140.97 85.6746 0)
+			(at 236.474 199.7206 0)
 			(show_name no)
 			(do_not_autoplace no)
@@
 			)
 		)
+		(pin "SCL" input
+			(at 111.76 38.1 0)
+			(effects
+				(font
+					(size 1.27 1.27)
+				)
+				(justify right)
+			)
+		)
+		(pin "SDA" input
+			(at 111.76 43.18 0)
+			(effects
+				(font
+					(size 1.27 1.27)
+				)
+				(justify right)
+			)
+		)
+		(pin "WRN" input
+			(at 111.76 46.99 0)
+			(effects
+				(font
+					(size 1.27 1.27)
+				)
+				(justify right)
+			)
+		)
 		(instances
 			(project "mach_robot"
@@
 			)
 		)
+		(pin "SCL" input
+			(at 238.76 54.61 180)
+			(effects
+				(font
+					(size 1.27 1.27)
+				)
+				(justify left)
+			)
+		)
+		(pin "SDA" input
+			(at 238.76 59.69 180)
+			(effects
+				(font
+					(size 1.27 1.27)
+				)
+				(justify left)
+			)
+		)
+		(pin "WRN" input
+			(at 238.76 66.04 180)
+			(effects
+				(font
+					(size 1.27 1.27)
+				)
+				(justify left)
+			)
+		)
