File: hardware/pcb/QUADRUPED_ROBOT/servo.kicad_sch (KiCad schematic)
At the start: 48 parts, among them J11 Conn_01x03_Pin, J12 Conn_01x03_Pin, J13 Conn_01x03_Pin, J14 Conn_01x03_Pin, J15 Conn_01x03_Pin, J16 Conn_01x03_Pin, J17 Conn_01x03_Pin, J18 Conn_01x03_Pin, J19 Conn_01x03_Pin, J20 Conn_01x03_Pin, J21 Conn_01x03_Pin, J22 Conn_01x03_Pin

Commit message: pcb update
Connections:
- net +6V renamed +6V_SERVO
Changed lines of the file:
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@@
 			)
 		)
-		(property "Value" "+6V"
+		(property "Value" "+6V_SERVO"
 			(at 46.99 151.1299 90)
 			(show_name no)
@@
 			)
 		)
-		(property "Value" "+6V"
+		(property "Value" "+6V_SERVO"
 			(at 55.88 72.3899 90)
 			(show_name no)
@@
 			)
 		)
-		(property "Value" "+6V"
+		(property "Value" "+6V_SERVO"
 			(at 55.88 31.7499 90)
 			(show_name no)
@@
 			)
 		)
-		(property "Value" "+6V"
+		(property "Value" "+6V_SERVO"
 			(at 139.7 106.6799 90)
 			(show_name no)
@@
 			)
 		)
-		(property "Value" "+6V"
+		(property "Value" "+6V_SERVO"
 			(at 142.24 68.5799 90)
 			(show_name no)
@@
 			)
 		)
-		(property "Value" "+6V"
+		(property "Value" "+6V_SERVO"
 			(at 44.45 130.8099 90)
 			(show_name no)
@@
 			)
 		)
-		(property "Value" "+6V"
+		(property "Value" "+6V_SERVO"
 			(at 53.34 52.0699 90)
 			(show_name no)
@@
 			)
 		)
-		(property "Value" "+6V"
+		(property "Value" "+6V_SERVO"
 			(at 139.7 48.2599 90)
 			(show_name no)
@@
 			)
 		)
-		(property "Value" "+6V"
+		(property "Value" "+6V_SERVO"
 			(at 139.7 147.3199 90)
 			(show_name no)
@@
 			)
 		)
-		(property "Value" "+6V"
+		(property "Value" "+6V_SERVO"
 			(at 46.99 110.4899 90)
 			(show_name no)
@@
 			)
 		)
-		(property "Value" "+6V"
+		(property "Value" "+6V_SERVO"
 			(at 137.16 126.9999 90)
 			(show_name no)
@@
 			)
 		)
-		(property "Value" "+6V"
+		(property "Value" "+6V_SERVO"
 			(at 142.24 27.9399 90)
 			(show_name no)
