Commit message: URDF fix

File: URDF/urdf/URDF.urdf (robot description, URDF)
Before this commit: robot URDF_1, 17 links, 16 joints
Links:
- removed link hip_LB
- removed link hip_LF
- removed link hip_RB
- added link Hip_LB, mass 0.0691271457278031; collision mesh filename=package://URDF/meshes/Hip_LB.STL; visual mesh filename=package://URDF/meshes/Hip_LB.STL
- added link Hip_LF, mass 0.069127; collision mesh filename=package://URDF/meshes/Hip_LF.STL; visual mesh filename=package://URDF/meshes/Hip_LF.STL
- added link Hip_RB, mass 0.0691271472886633; collision mesh filename=package://URDF/meshes/Hip_RB.STL; visual mesh filename=package://URDF/meshes/Hip_RB.STL
- link Calf_LB: mass 0.00886599097543008 -> 0.00886593782689565; geometry collision mesh filename=package://URDF/meshes/Calf_LB.STL; visual mesh filename=package://URDF/meshes/Calf_LB.STL
- link Calf_LF: mass 0.00886599216069642 -> 0.00886599216069837; geometry collision mesh filename=package://URDF/meshes/Calf_LF.STL; visual mesh filename=package://URDF/meshes/Calf_LF.STL
- link Calf_RB: mass 0.00886600238835241 -> 0.00886600305804803; geometry collision mesh filename=package://URDF/meshes/Calf_RB.STL; visual mesh filename=package://URDF/meshes/Calf_RB.STL
- link Calf_RF: mass 0.00886601403821351 -> 0.00886601436486069; geometry collision mesh filename=package://URDF/meshes/Calf_RF.STL; visual mesh filename=package://URDF/meshes/Calf_RF.STL
- link Foot_LB: mass 0.00230350113703878 -> 0.00230350113970975; geometry collision mesh filename=package://URDF/meshes/Foot_LB.STL; visual mesh filename=package://URDF/meshes/Foot_LB.STL
- link Foot_LF: mass 0.00230350113811289 -> 0.00230350113811287; geometry collision mesh filename=package://URDF/meshes/Foot_LF.STL; visual mesh filename=package://URDF/meshes/Foot_LF.STL
- link Foot_RB: mass 0.00230350114530592 -> 0.00230350114517015; geometry collision mesh filename=package://URDF/meshes/Foot_RB.STL; visual mesh filename=package://URDF/meshes/Foot_RB.STL
- link Foot_RF: mass 0.0023035 -> 0.00230350114254969; geometry collision mesh filename=package://URDF/meshes/Foot_RF.STL; visual mesh filename=package://URDF/meshes/Foot_RF.STL
- link Thigh_LB: mass 0.0136519260871885 -> 0.0136519261569896; geometry collision mesh filename=package://URDF/meshes/Thigh_LB.STL; visual mesh filename=package://URDF/meshes/Thigh_LB.STL
- link Thigh_LF: mass 0.0136519262084261 -> 0.013652; geometry collision mesh filename=package://URDF/meshes/Thigh_LF.STL; visual mesh filename=package://URDF/meshes/Thigh_LF.STL
- link Thigh_RB: mass 0.0136519260994358 -> 0.0136519261014922; geometry collision mesh filename=package://URDF/meshes/Thigh_RB.STL; visual mesh filename=package://URDF/meshes/Thigh_RB.STL
- link Thigh_RF: mass 0.0136519260754069 -> 0.013651926085773; geometry collision mesh filename=package://URDF/meshes/Thigh_RF.STL; visual mesh filename=package://URDF/meshes/Thigh_RF.STL
- link base_link: geometry collision mesh filename=package://URDF/meshes/base_link.STL; visual mesh filename=package://URDF/meshes/base_link.STL
- link hip_RF: mass 0 -> 0.0691270911282823; geometry collision mesh filename=package://URDF/meshes/hip_RF.STL; visual mesh filename=package://URDF/meshes/hip_RF.STL
Joints:
- joint Joint1_LB: axis 0 0 1 -> 0 0 -1; child hip_LB -> Hip_LB; origin xyz=0.045 0.095499 0.0093429 rpy=1.5708 1.5708 0 -> xyz=0.0449999975183657 0.0954992296169666 0.00938098015422961 rpy=-1.57079632679533 1.51781885809782 0
- joint Joint1_LF: axis 0 0 1 -> 0 0 -1; child hip_LF -> Hip_LF; origin xyz=0.0450000000000002 -0.0954992296169665 0.00934287444808674 rpy=1.5707963267949 1.5707963267949 0 -> xyz=0.045 -0.095499 0.009381 rpy=1.5708 1.5617 0
- joint Joint1_RB: axis 0 0 1 -> 0 0 -1; child hip_RB -> Hip_RB; origin xyz=-0.045 0.095499 0.0093429 rpy=-0.15362 1.5708 1.4441 -> xyz=-0.0450000024816331 0.0954992296169642 0.00938098015422933 rpy=-1.57079632679485 1.55110721336966 0
- joint Joint1_RF: axis 0 0 1 -> 0 0 -1; origin xyz=-0.0450000000000002 -0.095499229616963 0.00934287444808762 rpy=1.5707963267949 1.5707963267949 0 -> xyz=-0.0449999975183671 -0.0954992296169629 0.00938098015422906 rpy=1.5707963267949 1.5707963267949 0
- joint Joint2_LB: axis 0 0 1 -> 0 0 -1; origin xyz=0.0022793837699181 -0.0253982468305898 0.0398999999999235 rpy=1.5707963267949 0 0.0844627326260078 -> xyz=0.000166657436375506 -0.0254979846657288 0.0399381057240706 rpy=1.57079632679489 0 0; parent hip_LB -> Hip_LB
- joint Joint2_LF: axis 0 0 1 -> 0 0 -1; origin xyz=-0.000103830202143829 0.0255001128999754 0.0199 rpy=-1.5707963267949 0 0.00911492757548553 -> xyz=0.00016671 0.0255 0.019862 rpy=-1.5708 0 0; parent hip_LF -> Hip_LF
- joint Joint2_RB: axis 0 0 1 -> 0 0 -1; origin xyz=0.000334819020600619 0.0254981261046049 0.039899999999996 rpy=1.57079632679489 0 3.13350548107536 -> xyz=0.000166704579416199 0.0255007569262712 0.0399381047387575 rpy=-1.5707963267949 0 0; parent hip_RB -> Hip_RB
- joint Joint2_RF: axis 0 0 1 -> 0 0 -1; origin xyz=-0.00177477684565508 -0.0254384886691494 0.0198999999999995 rpy=1.5707963267949 0 -0.0746977131182892 -> xyz=-0.00173667361422397 -0.0254384909655809 0.0198618942938599 rpy=1.5707963267949 0 -0.0746977131182897
- joint Joint3_LB: axis 0 0 1 -> 0 0 -1; origin xyz=0.0814318538016524 0.058041822878408 0.0239000001044983 rpy=0 0 0 -> xyz=0.0809190598674842 0.0587165140777625 0.00130000001784963 rpy=0 0 0
- joint Joint3_LF: axis 0.0091148013617523 -0.1552882099193 -0.987827157075667 -> 0 0 -1; origin xyz=0.0899941947746462 0.0436009736916917 0.0238999999999975 rpy=0.155925725989217 0.0091149275754857 0 -> xyz=0.089994 0.043563 0.0013 rpy=0 0 0
- joint Joint3_RB: origin xyz=-0.0743002608384791 0.0669288520694507 0.0238999999999875 rpy=0 0 0 -> xyz=0.073521684021235 -0.0677450896688274 0.00129999081166665 rpy=0 0 0
- joint Joint3_RF: origin xyz=0.0780144504790948 -0.0625599353935496 0.0238999999999989 rpy=0 0 0 -> xyz=0.0805856649939703 -0.0591729658721312 0.00130000000000041 rpy=0 0 0
- joint Joint4_LB: origin xyz=0.096595 -0.068832 -0.012337 rpy=-3.0606 -1.5708 0.0023759 -> xyz=0.0849599453223677 -0.0827669358122232 0.0102631627484333 rpy=0 0 -0.0700282136507758
- joint Joint4_LF: origin xyz=0.09018 -0.078082 0.00027294 rpy=1.5067 -1.4146 1.6294 -> xyz=0.090068 -0.077177 0.0099224 rpy=0 0 -0.0061764
- joint Joint4_RB: origin xyz=-0.066585 -0.098158 -0.012678 rpy=0.25255 -1.5708 0.071307 -> xyz=0.0664620022781575 0.0982413366463415 0.00992243475666016 rpy=0 0 0.273708943903006
- joint Joint4_RF: origin xyz=0.084396 0.083342 -0.012322 rpy=0.076814 -1.5708 0 -> xyz=0.0849986200651742 0.0827272177698522 0.00992243475665372 rpy=0 0 0.0695608286554116
