Commit message: update URDF and cad

File: URDF_1/urdf/URDF_1.urdf (robot description, URDF)
Before this commit: robot final, 13 links, 12 joints
Links:
- added link Foot_LB, mass 0.00230350113703878; collision mesh filename=package://URDF_1/meshes/Foot_LB.STL; visual mesh filename=package://URDF_1/meshes/Foot_LB.STL
- added link Foot_LF, mass 0.00230350113811289; collision mesh filename=package://URDF_1/meshes/Foot_LF.STL; visual mesh filename=package://URDF_1/meshes/Foot_LF.STL
- added link Foot_RB, mass 0.00230350114530592; collision mesh filename=package://URDF_1/meshes/Foot_RB.STL; visual mesh filename=package://URDF_1/meshes/Foot_RB.STL
- added link Foot_RF, mass 0.0023035; collision mesh filename=package://URDF_1/meshes/Foot_RF.STL; visual mesh filename=package://URDF_1/meshes/Foot_RF.STL
- link Calf_LB: mass 0.00886599097543363 -> 0.00886599097543008; geometry collision mesh filename=package://URDF_1/meshes/Calf_LB.STL; visual mesh filename=package://URDF_1/meshes/Calf_LB.STL
- link Calf_LF: mass 0.00886599216069645 -> 0.00886599216069642; geometry collision mesh filename=package://URDF_1/meshes/Calf_LF.STL; visual mesh filename=package://URDF_1/meshes/Calf_LF.STL
- link Calf_RB: mass 0.00886600238835247 -> 0.00886600238835241; geometry collision mesh filename=package://URDF_1/meshes/Calf_RB.STL; visual mesh filename=package://URDF_1/meshes/Calf_RB.STL
- link Calf_RF: mass 0.00886601403821361 -> 0.00886601403821351; geometry collision mesh filename=package://URDF_1/meshes/Calf_RF.STL; visual mesh filename=package://URDF_1/meshes/Calf_RF.STL
- link Thigh_LB: geometry collision mesh filename=package://URDF_1/meshes/Thigh_LB.STL; visual mesh filename=package://URDF_1/meshes/Thigh_LB.STL
- link Thigh_LF: mass 0.0136519262084262 -> 0.0136519262084261; geometry collision mesh filename=package://URDF_1/meshes/Thigh_LF.STL; visual mesh filename=package://URDF_1/meshes/Thigh_LF.STL
- link Thigh_RB: mass 0.0136519260994359 -> 0.0136519260994358; geometry collision mesh filename=package://URDF_1/meshes/Thigh_RB.STL; visual mesh filename=package://URDF_1/meshes/Thigh_RB.STL
- link Thigh_RF: geometry collision mesh filename=package://URDF_1/meshes/Thigh_RF.STL; visual mesh filename=package://URDF_1/meshes/Thigh_RF.STL
- link base_link: geometry collision mesh filename=package://URDF_1/meshes/base_link.STL; visual mesh filename=package://URDF_1/meshes/base_link.STL
- link hip_LB: mass 0.0691271473745254 -> 0.0691271473763071; geometry collision mesh filename=package://URDF_1/meshes/hip_LB.STL; visual mesh filename=package://URDF_1/meshes/hip_LB.STL
- link hip_LF: mass 0.0691270861873928 -> 0.0691270851973415; geometry collision mesh filename=package://URDF_1/meshes/hip_LF.STL; visual mesh filename=package://URDF_1/meshes/hip_LF.STL
- link hip_RB: mass 0.0691271481987827 -> 0.0691271480360492; geometry collision mesh filename=package://URDF_1/meshes/hip_RB.STL; visual mesh filename=package://URDF_1/meshes/hip_RB.STL
- link hip_RF: mass 0.0691270910624313 -> 0; geometry collision mesh filename=package://URDF_1/meshes/hip_RF.STL; visual mesh filename=package://URDF_1/meshes/hip_RF.STL
Joints:
- added joint Joint4_LB: type fixed, parent Calf_LB, child Foot_LB, origin xyz=0.096595 -0.068832 -0.012337 rpy=-3.0606 -1.5708 0.0023759, axis 0 0 0
- added joint Joint4_LF: type fixed, parent Calf_LF, child Foot_LF, origin xyz=0.09018 -0.078082 0.00027294 rpy=1.5067 -1.4146 1.6294, axis 0 0 0
- added joint Joint4_RB: type fixed, parent Calf_RB, child Foot_RB, origin xyz=-0.066585 -0.098158 -0.012678 rpy=0.25255 -1.5708 0.071307, axis 0 0 0
- added joint Joint4_RF: type fixed, parent Calf_RF, child Foot_RF, origin xyz=0.084396 0.083342 -0.012322 rpy=0.076814 -1.5708 0, axis 0 0 0
- joint Joint1_LB: origin xyz=0.256926339687758 -0.50176821300437 0.220696871077039 rpy=2.43571062058662 1.04313880299812 2.52448464320818 -> xyz=0.045 0.095499 0.0093429 rpy=1.5708 1.5708 0
- joint Joint1_LF: origin xyz=0.0828037089815861 -0.530142263822002 0.293885901306255 rpy=-0.705882033003174 1.04313880299812 2.52448464320818 -> xyz=0.0450000000000002 -0.0954992296169665 0.00934287444808674 rpy=1.5707963267949 1.5707963267949 0
- joint Joint1_RB: origin xyz=0.255423331114134 -0.416717792411357 0.250093587257239 rpy=2.43571062058662 1.04313880299812 2.52448464320818 -> xyz=-0.045 0.095499 0.0093429 rpy=-0.15362 1.5708 1.4441
- joint Joint1_RF: origin xyz=0.081301 -0.44509 0.32328 rpy=-0.70588 1.0431 2.5245 -> xyz=-0.0450000000000002 -0.095499229616963 0.00934287444808762 rpy=1.5707963267949 1.5707963267949 0
- joint Joint2_RF: origin xyz=-0.0017748 -0.025438 0.0199 rpy=1.5708 0 -0.074698 -> xyz=-0.00177477684565508 -0.0254384886691494 0.0198999999999995 rpy=1.5707963267949 0 -0.0746977131182892
- joint Joint3_LB: origin xyz=0.0814318625004756 0.0580418106742034 0.0239000001006261 rpy=0 0 0 -> xyz=0.0814318538016524 0.058041822878408 0.0239000001044983 rpy=0 0 0
- joint Joint3_LF: axis 0.00911480136175463 -0.155288209919299 -0.987827157075667 -> 0.0091148013617523 -0.1552882099193 -0.987827157075667
- joint Joint3_RF: origin xyz=0.078014 -0.06256 0.0239 rpy=0 0 0 -> xyz=0.0780144504790948 -0.0625599353935496 0.0238999999999989 rpy=0 0 0

Commit message: : URDF_1 recheck

File: URDF_1/urdf/URDF_1.urdf (robot description, URDF)
Before this commit: robot URDF_1, 17 links, 16 joints
Links:
- link Calf_LB: mass 0.00886599176378451 -> 0.00886598317933579
- link Calf_LF: mass 0.00886599233857974 -> 0.00886599012842122
- link Calf_RB: mass 0.00886600450407864 -> 0.008866
- link Calf_RF: mass 0.00886601522787845 -> 0.00886601726386029
- link Foot_LB: mass 0.00230350113779985 -> 0.0023035011249116
- link Foot_LF: mass 0.00230350113749122 -> 0.00230350113544803
- link Foot_RB: mass 0.00230350114512336 -> 0.0023035
- link Foot_RF: mass 0.00230350114184203 -> 0.00230350113995821
- link Hip_LB: mass 0.0691271451331567 -> 0.0691271600080189
- link Hip_LF: mass 0 -> 0.069127
- link Hip_RB: mass 0.069127145268005 -> 0.0691271608115489
- link Thigh_LB: mass 0.013652 -> 0.0136519259715228
- link Thigh_LF: mass 0.0136519261330692 -> 0.0136519261108968
- link Thigh_RB: mass 0.0136519260992832 -> 0.0136519260678425
- link Thigh_RF: mass 0.0136519261061882 -> 0.0136519261065869
- link base_link: mass 0.32654744983969 -> 0.326547450453838
- link hip_RF: mass 0.0691270911890896 -> 0.0691270950351537
Joints:
- joint Joint1_LB: origin xyz=0.0449999967362847 0.0954992300103887 0.009380981274699 rpy=1.57079628324533 1.40431060818658 3.14159260942963 -> xyz=0.0449999975824225 0.0954992295412814 0.00938097942002192 rpy=1.57079632495153 1.34679897174749 3.14159265169919
- joint Joint1_LF: origin xyz=0.0450000009972144 -0.0954992292242923 0.00938098007435328 rpy=-1.57079649690177 1.52835768215523 3.14159248242334 -> xyz=0.045 -0.095499 0.009381 rpy=-1.5708 1.4693 3.1416
- joint Joint1_RB: origin xyz=-0.0450000037192648 0.0954992301195679 0.00938098156076461 rpy=1.57079610030804 1.53892626120084 3.14159242600521 -> xyz=-0.045 0.095499 0.009381 rpy=1.5708 1.4798 3.1416
- joint Joint1_RF: origin xyz=-0.0449999990053749 -0.0954992291155026 0.00938098000774029 rpy=1.57079632800763 1.5707963267949 0 -> xyz=-0.0449999975183673 -0.0954992296169646 0.00938098015422839 rpy=1.5707963267949 1.5707963267949 0
- joint Joint2_LB: origin xyz=0.000166183759488514 -0.0255063180457349 0.0399381057123354 rpy=1.5707963267949 0 0 -> xyz=0.000165754722025624 -0.0255084660262564 0.039938106153917 rpy=1.5707963267949 0 0
- joint Joint2_LF: origin xyz=0.000166676854179038 0.0255016149609894 0.0198618943495757 rpy=-1.5707963267949 0 0 -> xyz=0.000166513432114379 0.0255038634633682 0.0198618913914449 rpy=-1.57079632679489 0 0
- joint Joint2_RB: origin xyz=0.00016669 0.025499 0.039938 rpy=-1.5708 0 0 -> xyz=0.000166547789723137 0.025496533420395 0.0399381057061415 rpy=-1.5707963267949 0 0
- joint Joint2_RF: origin xyz=-0.00304406186672296 -0.0253133727377505 0.0198618943689335 rpy=1.5707963267949 0 -0.126207137233731 -> xyz=-0.00450651591222284 -0.025092092493153 0.0198618938454757 rpy=1.5707963268116 0 -0.184218403881293
- joint Joint3_LB: origin xyz=0.0997055503615685 0.00763018747714993 0.00130000001065278 rpy=0 0 0 -> xyz=0.0972627533996326 0.0231988662333634 0.00129999934280145 rpy=0 0 0
- joint Joint3_LF: origin xyz=0.091508608335129 0.040287743110421 0.00130000035955524 rpy=0 0 0 -> xyz=0.0849262922412908 0.0527589116011191 0.00129999273078008 rpy=0 0 0
- joint Joint3_RB: origin xyz=0.0704636394572004 -0.0709187536109075 0.00130000022489368 rpy=0 0 0 -> xyz=0.0408860054507293 -0.0912215931263758 0.00130000120269708 rpy=0 0 0
- joint Joint3_RF: origin xyz=0.0826731320829293 -0.0562215942551578 0.00130000015939194 rpy=0 0 0 -> xyz=0.0732205350882606 -0.0680702904138538 0.00129999939815947 rpy=0 0 0
- joint Joint4_LB: origin xyz=0.0987143958873673 -0.0657573267211811 0.0102631627484327 rpy=0 0 0.114659882597004 -> xyz=0.118550160948996 -0.0037969819877507 0.0102631639512074 rpy=0 0 0.670278242890864
- joint Joint4_LF: origin xyz=0.0936058345991075 -0.072845766534023 0.00992243475665627 rpy=0 0 0.0409782674287381 -> xyz=0.106733851654356 -0.0517343491691078 0.00992243475665783 rpy=0 0 0.250959525591169
- joint Joint4_RB: origin xyz=0.0700973869395912 0.0956813164477049 0.00992243475665266 rpy=0 0 0.236220194369359 -> xyz=0.0821911036658188 0.0855171354239601 0.00992243475665383 rpy=0 0 0.102932003324284
- joint Joint4_RF: origin xyz=0.0891649502501446 0.0782187293415921 0.00992243475665497 rpy=0 0 0.0177993522340094 -> xyz=0.103568272218062 0.0578115123715837 0.00992243475665355 rpy=0 0 -0.193181008175667
